Commit message: typo xacro file

File: src/yambot/urdf/test_robot.xacro (robot description, xacro)
@@ -27,5 +27,5 @@
 		</collision>
 		<inertial>
-			<origion rpy="0 0 0" xyz="0 0 0" />
+			<origin rpy="0 0 0" xyz="0 0 0" />
 			<mass value="1"/>
 			<inertia ixx="100" ixy="0" ixz="0" iyy="100" iyz="0" izz="100" />
