Commit message: visible now in rviz

File: src/yambot/urdf/lidar.xacro (robot description, xacro)
@@ -6,4 +6,8 @@
     <xacro:property name="laser_height" value="0.175"/>
     <xacro:property name="laser_mass" value="0.1"/>
+    <!-- Define the material for the LiDAR -->
+    <material name="red">
+        <color rgba="1 0 0 1"/> <!-- Define the red material with full opacity -->
+    </material>
     <!-- This macro defines the complete inertial section of the LiDAR -->
     <xacro:macro name="inertial_laser">
@@ -24,5 +28,5 @@
                 <cylinder radius="${laser_radius}" length="${laser_length}"/>
             </geometry>
-            <material name="red"/>
+            <material name="red"/> <!-- Use the defined material -->
         </visual>
         <collision>
@@ -39,5 +43,5 @@
     </joint>
     <gazebo reference="laser_frame">
-        <material>Gazebo/Red</material>
+        <material>Gazebo/Red</material> <!-- Ensure the material is correctly referenced -->
         <sensor name="laser" type="ray">
             <pose>0 0 0 0 0 0</pose>

Commit message: slam not functioning correctly yet

File: src/yambot/urdf/lidar.xacro (robot description, xacro)
@@ -7,6 +7,6 @@
     <xacro:property name="laser_mass" value="0.1"/>
     <!-- Define the material for the LiDAR -->
-    <material name="red">
-        <color rgba="1 0 0 1"/> <!-- Define the red material with full opacity -->
+    <material name="yellow">
+    	<color rgba="1 1 0 1"/> <!-- Define the yellow material with full opacity -->
     </material>
     <!-- This macro defines the complete inertial section of the LiDAR -->
@@ -28,5 +28,5 @@
                 <cylinder radius="${laser_radius}" length="${laser_length}"/>
             </geometry>
-            <material name="red"/> <!-- Use the defined material -->
+            <material name="yellow"/> <!-- Use the defined material -->
         </visual>
         <collision>
@@ -43,5 +43,5 @@
     </joint>
     <gazebo reference="laser_frame">
-        <material>Gazebo/Red</material> <!-- Ensure the material is correctly referenced -->
+        <material>Gazebo/Yellow</material> <!-- Ensure the material is correctly referenced -->
         <sensor name="laser" type="ray">
             <pose>0 0 0 0 0 0</pose>
@@ -63,5 +63,5 @@
             <plugin name="laser_controller" filename="libgazebo_ros_ray_sensor.so">
                 <ros>
-                    <argument>~/out:=scan</argument>
+                    <argument>--ros-args --remap ~/out:=scan</argument>
                 </ros>
                 <output_type>sensor_msgs/LaserScan</output_type>
